File: HW/ELKS/ui.kicad_sch (KiCad schematic)
At the start: 30 parts, among them Q1 Q_NMOS_GSD, SW1 SW, SW2 SW, SW3 SW

Commit message: Fix potentiometers footprints and relocation of two component
Parts:
- RV1, RV2: footprint Potentiometer_THT:Potentiometer_Alpha_RD901F-40-00D_Single_Vertical -> Robotarna_KiCad_Library:RK09K113 (ELKS-POT)
Changed lines of the file:
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@@
       (effects (font (size 1.27 1.27)) (justify right))
     )
-    (property "Footprint" "Potentiometer_THT:Potentiometer_Alpha_RD901F-40-00D_Single_Vertical" (id 2) (at 139.7 92.71 0)
+    (property "Footprint" "Robotarna_KiCad_Library:RK09K113 (ELKS-POT)" (id 2) (at 139.7 92.71 0)
       (effects (font (size 1.27 1.27)) hide)
     )
@@
       (effects (font (size 1.27 1.27)) (justify right))
     )
-    (property "Footprint" "Potentiometer_THT:Potentiometer_Alpha_RD901F-40-00D_Single_Vertical" (id 2) (at 139.7 130.81 0)
+    (property "Footprint" "Robotarna_KiCad_Library:RK09K113 (ELKS-POT)" (id 2) (at 139.7 130.81 0)
       (effects (font (size 1.27 1.27)) hide)
     )
